File: IEE.kicad_pcb (KiCad board)
At the start: 2 copper layers, 333.4 x 95.2 mm, 195 parts, among them J1 JST 4 Pin, J2 AVR-ISP-6, J3 Conn_01x02_Male, Q1 TIP120, SW1 SW_Push, U1 ATmega32U4-A, U10 WS2812-2020, U11 WS2812-2020, U12 WS2812-2020, U13 WS2812-2020, U14 WS2812-2020, U15 WS2812-2020, U16 WS2812-2020, U17 WS2812-2020, U18 WS2812-2020, U19 WS2812-2020, U2 SRV05-4, U20 WS2812-2020, U21 WS2812-2020, U22 WS2812-2020, U23 WS2812-2020, U24 WS2812-2020, U25 WS2812-2020, U26 WS2812-2020, U3 WS2812-2020, U4 WS2812-2020, U5 WS2812-2020, U6 WS2812-2020, U7 WS2812-2020, U8 WS2812-2020, U9 WS2812-2020, Y1 16MHz

Commit message: Add Firmware VIAL and QMK in IEE-Firmware folder
Connections:
- MX74 pad 1: COL7 -> COL8
Changed lines of the file:
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@@
   (net 140 "Net-(Q1-PadB)")
   (net 141 "SOL")
+  (net 142 "COL8")
   (footprint "MX_Only:MXOnly-1U-NoLED" (layer "F.Cu")
     (at 204.7875 57.15)
@@
     (pad "" np_thru_hole circle locked (at 0 0) (size 3.9878 3.9878) (drill 3.9878) (layers *.Cu *.Mask))
     (pad "1" thru_hole circle locked (at -3.81 -2.54) (size 2.25 2.25) (drill 1.47) (layers *.Cu "B.Mask")
-      (net 102 "COL7") (pinfunction "COL") (pintype "passive"))
+      (net 142 "COL8") (pinfunction "COL") (pintype "passive"))
     (pad "2" thru_hole circle locked (at 2.54 -5.08) (size 2.25 2.25) (drill 1.47) (layers *.Cu "B.Mask")
       (net 112 "Net-(D74-Pad2)") (pinfunction "ROW") (pintype "passive"))
