File: IEE.kicad_sch (KiCad schematic)
At the start: 195 parts, among them J1 JST 4 Pin, J2 AVR-ISP-6, J3 Conn_01x02_Male, Q1 TIP120, SW1 SW_Push, U1 ATmega32U4-A, U10 WS2812-2020, U11 WS2812-2020, U12 WS2812-2020, U13 WS2812-2020, U14 WS2812-2020, U15 WS2812-2020, U16 WS2812-2020, U17 WS2812-2020, U18 WS2812-2020, U19 WS2812-2020, U2 SRV05-4, U20 WS2812-2020, U21 WS2812-2020, U22 WS2812-2020, U23 WS2812-2020, U24 WS2812-2020, U25 WS2812-2020, U26 WS2812-2020, U3 WS2812-2020, U4 WS2812-2020, U5 WS2812-2020, U6 WS2812-2020, U7 WS2812-2020, U8 WS2812-2020, U9 WS2812-2020, Y1 16MHz

Commit message: Add Firmware VIAL and QMK in IEE-Firmware folder
Connections:
- net COL7: no longer MX74.1 (COL)
- new net COL8: MX74.1 (COL)
Changed lines of the file:
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@@
   (junction (at 177.8 33.02) (diameter 0) (color 0 0 0 0)
   )
-  (junction (at 317.5 25.4) (diameter 0) (color 0 0 0 0)
-  )
   (junction (at 558.8 122.555) (diameter 0) (color 0 0 0 0)
   )
@@
   )
   (wire (pts (xy 28.575 40.64) (xy 41.91 40.64))
-    (stroke (width 0) (type default) (color 0 0 0 0))
-  )
-  (wire (pts (xy 317.5 25.4) (xy 330.2 25.4))
     (stroke (width 0) (type default) (color 0 0 0 0))
   )
@@
     )
   )
+  (global_label "COL8" (shape input) (at 330.2 25.4 90) (fields_autoplaced)
+    (effects (font (size 1.27 1.27)) (justify left))
+    (property "Intersheet References" "${INTERSHEET_REFS}" (id 0) (at 330.1206 18.1488 90)
+      (effects (font (size 1.27 1.27)) (justify left) hide)
+    )
+  )
   (global_label "SCK" (shape input) (at 43.815 143.51 0) (fields_autoplaced)
     (effects (font (size 1.27 1.27)) (justify left))
@@
       (effects (font (size 1.27 1.27)) (justify left) hide)
     )
+  )
+  (global_label "COL8" (shape input) (at -172.085 86.995 0) (fields_autoplaced)
+    (effects (font (size 1.27 1.27)) (justify left))
+    (property "Intersheet References" "${INTERSHEET_REFS}" (id 0) (at -164.8338 86.9156 0)
+      (effects (font (size 1.27 1.27)) (justify left) hide)
+    )
